Commit message: Working icp_odometry + RTABMap SLAM - LiDAR TF calibrated
- icp_odometry replaces point_lio - no timestamp issues, built-in IMU support
- Removed static lidar TF from launch file - XACRO is sole authority
- LiDAR yaw calibrated to 72 degrees (1.2566 rad) counterclockwise from forward
- IMU gravity alignment via wait_imu_to_init
- cloud_subtract_filtering enabled
- RGBD/LinearUpdate and AngularUpdate 0.1 to reduce stationary drift

File: urdf/tank_robot.xacro (robot description, xacro)
@@ -132,5 +132,5 @@
     <parent link="base_link"/>
     <child link="lidar_link"/>
-    <origin xyz="0.15 0 0.50" rpy="0 0 1.9199"/>
+    <origin xyz="0.15 0 0.50" rpy="0 0 1.2566"/>
   </joint>
   <link name="unilidar_lidar"/>

Commit message: urdf: apply calibrated lidar_joint extrinsic transform
rpy: 0 0 1.2566 (visual yaw only) -> 0.360 0.215 1.273 (calibrated)

File: urdf/tank_robot.xacro (robot description, xacro)
@@ -132,5 +132,5 @@
     <parent link="base_link"/>
     <child link="lidar_link"/>
-    <origin xyz="0.15 0 0.50" rpy="0 0 1.2566"/>
+    <origin xyz="0.15 0 0.50" rpy="0.360 0.215 1.273"/>
   </joint>
   <link name="unilidar_lidar"/>
